Commit message: tried adding four bar linkage sdf and visualizing in gazebo, did not work

File: finger_description/urdf/finger.urdf.xacro (robot description, xacro)
@@ -1,5 +1,5 @@
 <?xml version="1.0"?>
 <robot name="finger">
-  <!-- Generated by urdf_blender_export.py from Blender scene /home/michael-jenz/rds_ws/finger_vizualization/src/blender_files/rds_finger.blend -->
+  <!-- Generated by urdf_blender_export.py from Blender scene /home/michael-jenz/rds_ws/finger_vizualization/src/drake-finger-sim/blender_files/rds_finger2.blend -->
   <material name="blue">
     <color rgba="0 0 1 1"/>
@@ -42,5 +42,5 @@
     <parent link="base_link"/>
     <child link="mcp_link"/>
-    <origin xyz="-0.0 1.3926 0.6693" rpy="0 0 0"/>
+    <origin xyz="0.0 0.0196 0.017" rpy="0 0 0"/>
     <axis xyz="0.0 0.0 1.0"/>
     <limit lower="-0.174533" upper="0.174533" effort="5.0" velocity="3.14"/>
@@ -69,7 +69,7 @@
     <parent link="mcp_link"/>
     <child link="proximal_phalanx"/>
-    <origin xyz="-0.0012 0.6999 0.0" rpy="0 0 0"/>
-    <axis xyz="1.0 0.0 0.0"/>
-    <limit lower="-1.57" upper="0.0" effort="5.0" velocity="3.14"/>
+    <origin xyz="-0.0 0.0177 0.0" rpy="0 0 0"/>
+    <axis xyz="-1.0 0.0 0.0"/>
+    <limit lower="0.0" upper="1.57" effort="5.0" velocity="3.14"/>
     <dynamics damping="0.1" friction="0.05"/>
   </joint>
@@ -96,7 +96,7 @@
     <parent link="proximal_phalanx"/>
     <child link="middle_phalanx"/>
-    <origin xyz="-0.0042 2.4094 0.0" rpy="0 0 0"/>
-    <axis xyz="1.0 0.0 0.0"/>
-    <limit lower="-1.57" upper="0.0" effort="5.0" velocity="3.14"/>
+    <origin xyz="-0.0001 0.0612 -0.0017" rpy="0 0 0"/>
+    <axis xyz="-1.0 0.0 0.0"/>
+    <limit lower="0.0" upper="1.57" effort="5.0" velocity="3.14"/>
     <dynamics damping="0.1" friction="0.05"/>
   </joint>
@@ -123,7 +123,7 @@
     <parent link="middle_phalanx"/>
     <child link="distal_phalanx"/>
-    <origin xyz="0.139 1.5987 0.0" rpy="0 0 0"/>
-    <axis xyz="1.0 0.0 0.0"/>
-    <limit lower="-1.57" upper="0.0" effort="3.0" velocity="3.14"/>
+    <origin xyz="0.0036 0.0406 -0.0023" rpy="0 0 0"/>
+    <axis xyz="-1.0 0.0 0.0"/>
+    <limit lower="0.0" upper="1.57" effort="3.0" velocity="3.14"/>
     <dynamics damping="0.1" friction="0.05"/>
     <mimic joint="pip_flexion" multiplier="0.85" offset="0.0"/>
