Commit message: cleaned up code, removed 4 bar linkage attempt

File: finger_description/urdf/finger.urdf (robot description, URDF)
Before this commit: robot finger, 5 links, 4 joints
Joints:
- joint mcp_flexion: limit lower=0.0 upper=1.57 effort=5.0 velocity=3.14 -> lower=0 upper=1.57 effort=5.0 velocity=3.14

Commit message: implemented mass and inertia calculation from blender into sdf

File: finger_description/urdf/finger.urdf (robot description, URDF)
Before this commit: robot finger, 5 links, 4 joints
Links:
- link base_link: geometry collision mesh filename=package://finger_description/meshes/urdf/collision/col_base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; visual mesh filename=package://finger_description/meshes/urdf/visual/base_link.o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
- link distal_phalanx: geometry collision mesh filename=package://finger_description/meshes/urdf/collision/col_dist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; visual mesh filename=package://finger_description/meshes/urdf/visual/distal_phal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
- link mcp_link: geometry collision mesh filename=package://finger_description/meshes/urdf/collision/col_mcp_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; visual mesh filename=package://finger_description/meshes/urdf/visual/mcp_link.obj
- link middle_phalanx: geometry collision mesh filename=package://finger_description/meshes/urdf/collision/col_midd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; visual mesh filename=package://finger_description/meshes/urdf/visual/middle_phal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
- link proximal_phalanx: geometry collision mesh filename=package://finger_description/meshes/urdf/collision/col_prox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; visual mesh filename=package://finger_description/meshes/urdf/visual/proximal_ph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
